File: kicad/DigitalVFO/DigitalVFO.sch (KiCad schematic (older format))
At the start: 23 parts, among them J1 Coax, J2 Conn_01x03, Q1 2N2222A, SW1 Rotary_Encoder_Switch, U1 74HC14, U2 Teensy3.2, U3 LCD1602A, U4 DDS-60

Commit message: Changing footprints and smaller board
Parts:
- U3: footprint (none) -> teensy:Conn_LCD16
- U4: footprint (none) -> teensy:Conn_DDS8
Changed lines of the file:
@@
 F 0 "U4" H 5750 6000 60  0000 C CNN
 F 1 "DDS-60" H 6600 5550 60  0000 C CNN
-F 2 "" H 6600 5550 60  0001 C CNN
+F 2 "teensy:Conn_DDS8" H 6600 5550 60  0001 C CNN
 F 3 "" H 6600 5550 60  0001 C CNN
 	1    6600 5550
@@
 F 0 "U3" H 7950 3700 60  0000 C CNN
 F 1 "LCD1602A" H 8250 2700 60  0000 C CNN
-F 2 "" H 8250 2900 60  0001 C CNN
+F 2 "teensy:Conn_LCD16" H 8250 2900 60  0001 C CNN
 F 3 "" H 8250 2900 60  0001 C CNN
 	1    8250 2900

Commit message: Working on new PCB
Parts:
- J1: footprint teensy:Conn_SMA_Edge -> Connectors:SMA_THT_Jack_Straight
Changed lines of the file:
@@
 F 0 "J1" V 7000 4500 50  0000 C CNN
 F 1 "Coax" V 7000 4350 50  0000 C CNN
-F 2 "teensy:Conn_SMA_Edge" H 6900 4450 50  0001 C CNN
+F 2 "Connectors:SMA_THT_Jack_Straight" H 6900 4450 50  0001 C CNN
 F 3 "" H 6900 4450 50  0001 C CNN
 	1    6900 4450

Commit message: Almost ready with v1.2
Parts:
- removed J2: Conn_01x03, teensy:Conn_Power_3, symbol Conn_01x03
- added C6, C7: 0.1uF, teensy:Cap_SmV, symbol C_Small
- added J2: Conn_01x02, teensy:Conn_Power_2, symbol Conn_01x02
- J1: footprint Connectors:SMA_THT_Jack_Straight -> teensy:BNC_Socket
- U2: footprint teensy:Conn_DIP28w -> (none)
- U3: footprint teensy:Conn_LCD16 -> (none)
Connections:
- wire segments 55 -> 54
Changed lines of the file:
@@
 F 0 "J1" V 7000 4500 50  0000 C CNN
 F 1 "Coax" V 7000 4350 50  0000 C CNN
-F 2 "Connectors:SMA_THT_Jack_Straight" H 6900 4450 50  0001 C CNN
+F 2 "teensy:BNC_Socket" H 6900 4450 50  0001 C CNN
 F 3 "" H 6900 4450 50  0001 C CNN
 	1    6900 4450
 	0    -1   -1   0
 $EndComp
-Wire Wire Line
-	6600 4950 6600 4700
 Wire Wire Line
 	3650 2750 3650 2700
@@
 $Comp
 L GND #PWR04
-U 1 1 5A324DF6
-P 8000 5050
-F 0 "#PWR04" H 8000 4800 50  0001 C CNN
-F 1 "GND" H 8000 4900 50  0000 C CNN
-F 2 "" H 8000 5050 50  0001 C CNN
-F 3 "" H 8000 5050 50  0001 C CNN
-	1    8000 5050
-	1    0    0    -1
-$EndComp
-$Comp
-L GND #PWR05
 U 1 1 5A32516D
 P 3650 3600
-F 0 "#PWR05" H 3650 3350 50  0001 C CNN
+F 0 "#PWR04" H 3650 3350 50  0001 C CNN
 F 1 "GND" H 3650 3450 50  0000 C CNN
 F 2 "" H 3650 3600 50  0001 C CNN
@@
 $EndComp
 $Comp
-L GND #PWR06
+L GND #PWR05
 U 1 1 5A325232
 P 2800 2650
-F 0 "#PWR06" H 2800 2400 50  0001 C CNN
+F 0 "#PWR05" H 2800 2400 50  0001 C CNN
 F 1 "GND" H 2800 2500 50  0000 C CNN
 F 2 "" H 2800 2650 50  0001 C CNN
@@
 $EndComp
 $Comp
-L GND #PWR07
+L GND #PWR06
 U 1 1 5A32532D
 P 6950 3200
-F 0 "#PWR07" H 6950 2950 50  0001 C CNN
+F 0 "#PWR06" H 6950 2950 50  0001 C CNN
 F 1 "GND" H 6950 3050 50  0000 C CNN
 F 2 "" H 6950 3200 50  0001 C CNN
@@
 $EndComp
 $Comp
-L GND #PWR08
+L GND #PWR07
 U 1 1 5A325451
 P 8350 3850
-F 0 "#PWR08" H 8350 3600 50  0001 C CNN
+F 0 "#PWR07" H 8350 3600 50  0001 C CNN
 F 1 "GND" H 8350 3700 50  0000 C CNN
 F 2 "" H 8350 3850 50  0001 C CNN
@@
 $EndComp
 $Comp
-L GND #PWR09
+L GND #PWR08
 U 1 1 5A325545
 P 5600 3950
-F 0 "#PWR09" H 5600 3700 50  0001 C CNN
+F 0 "#PWR08" H 5600 3700 50  0001 C CNN
 F 1 "GND" H 5600 3800 50  0000 C CNN
 F 2 "" H 5600 3950 50  0001 C CNN
@@
 $EndComp
 $Comp
-L GND #PWR010
+L GND #PWR09
 U 1 1 5A32580E
 P 6750 4900
-F 0 "#PWR010" H 6750 4650 50  0001 C CNN
+F 0 "#PWR09" H 6750 4650 50  0001 C CNN
 F 1 "GND" H 6750 4750 50  0000 C CNN
 F 2 "" H 6750 4900 50  0001 C CNN
@@
 $EndComp
 $Comp
-L GND #PWR011
+L GND #PWR010
 U 1 1 5A32593F
 P 7150 4050
-F 0 "#PWR011" H 7150 3800 50  0001 C CNN
+F 0 "#PWR010" H 7150 3800 50  0001 C CNN
 F 1 "GND" H 7150 3900 50  0000 C CNN
 F 2 "" H 7150 4050 50  0001 C CNN
@@
 $EndComp
 $Comp
-L GND #PWR012
+L GND #PWR011
 U 1 1 5A325A73
 P 3950 5600
-F 0 "#PWR012" H 3950 5350 50  0001 C CNN
+F 0 "#PWR011" H 3950 5350 50  0001 C CNN
 F 1 "GND" H 3950 5450 50  0000 C CNN
 F 2 "" H 3950 5600 50  0001 C CNN
@@
 $EndComp
 $Comp
-L GND #PWR013
+L GND #PWR012
 U 1 1 5A325F7B
 P 7100 4450
-F 0 "#PWR013" H 7100 4200 50  0001 C CNN
+F 0 "#PWR012" H 7100 4200 50  0001 C CNN
 F 1 "GND" H 7100 4300 50  0000 C CNN
 F 2 "" H 7100 4450 50  0001 C CNN
@@
 $EndComp
 $Comp
-L +5V #PWR014
+L +5V #PWR013
 U 1 1 5A327357
 P 5950 1750
-F 0 "#PWR014" H 5950 1600 50  0001 C CNN
+F 0 "#PWR013" H 5950 1600 50  0001 C CNN
 F 1 "+5V" H 5950 1890 50  0000 C CNN
 F 2 "" H 5950 1750 50  0001 C CNN
@@
 $EndComp
 $Comp
-L +5V #PWR015
+L +5V #PWR014
 U 1 1 5A327500
 P 3650 2700
-F 0 "#PWR015" H 3650 2550 50  0001 C CNN
+F 0 "#PWR014" H 3650 2550 50  0001 C CNN
 F 1 "+5V" H 3650 2840 50  0000 C CNN
 F 2 "" H 3650 2700 50  0001 C CNN
@@
 $EndComp
 $Comp
-L +5V #PWR016
+L +5V #PWR015
 U 1 1 5A327580
 P 3200 3600
-F 0 "#PWR016" H 3200 3450 50  0001 C CNN
+F 0 "#PWR015" H 3200 3450 50  0001 C CNN
 F 1 "+5V" H 3200 3740 50  0000 C CNN
 F 2 "" H 3200 3600 50  0001 C CNN
@@
 Connection ~ 7150 1750
 $Comp
-L VCC #PWR017
+L VCC #PWR016
 U 1 1 5A327A0A
 P 7150 1750
-F 0 "#PWR017" H 7150 1600 50  0001 C CNN
+F 0 "#PWR016" H 7150 1600 50  0001 C CNN
 F 1 "VCC" H 7150 1900 50  0000 C CNN
 F 2 "" H 7150 1750 50  0001 C CNN
@@
 $EndComp
 $Comp
-L VCC #PWR018
+L VCC #PWR017
 U 1 1 5A3280F4
-P 6600 4700
-F 0 "#PWR018" H 6600 4550 50  0001 C CNN
-F 1 "VCC" H 6600 4850 50  0000 C CNN
-F 2 "" H 6600 4700 50  0001 C CNN
-F 3 "" H 6600 4700 50  0001 C CNN
-	1    6600 4700
-	1    0    0    -1
-$EndComp
-Wire Wire Line
-	7200 4950 8100 4950
-Wire Wire Line
-	8100 4850 8000 4850
-Wire Wire Line
-	8000 4850 8000 5050
-Wire Wire Line
-	8000 5050 8100 5050
-$Comp
-L Conn_01x03 J2
-U 1 1 5A32F0C2
-P 8300 4950
-F 0 "J2" H 8300 5150 50  0000 C CNN
-F 1 "Conn_01x03" V 8400 4950 31  0000 C CNN
-F 2 "teensy:Conn_Power_3" H 8300 4950 50  0001 C CNN
-F 3 "" H 8300 4950 50  0001 C CNN
-	1    8300 4950
+P 6600 4550
+F 0 "#PWR017" H 6600 4400 50  0001 C CNN
+F 1 "VCC" H 6600 4700 50  0000 C CNN
+F 2 "" H 6600 4550 50  0001 C CNN
+F 3 "" H 6600 4550 50  0001 C CNN
+	1    6600 4550
 	1    0    0    -1
 $EndComp
@@
 $EndComp
 $Comp
-L GND #PWR019
+L GND #PWR018
 U 1 1 5A3E323F
 P 6200 2000
-F 0 "#PWR019" H 6200 1750 50  0001 C CNN
+F 0 "#PWR018" H 6200 1750 50  0001 C CNN
 F 1 "GND" H 6350 1950 50  0000 C CNN
 F 2 "" H 6200 2000 50  0001 C CNN
@@
 $EndComp
 Connection ~ 6200 1750
-$Comp
-L Teensy3.2 U2
-U 1 1 5A446CDC
-P 5950 2950
-F 0 "U2" H 5600 3800 60  0000 C CNN
-F 1 "Teensy3.2" H 5950 2950 60  0000 C CNN
-F 2 "teensy:Conn_DIP28w" H 5950 2950 60  0001 C CNN
-F 3 "" H 5950 2950 60  0001 C CNN
-	1    5950 2950
-	1    0    0    -1
-$EndComp
 Wire Wire Line
 	6200 1800 6200 1750
@@
 	1    0    0    -1
 $EndComp
+Wire Wire Line
+	2900 2050 4100 2050
+Wire Wire Line
+	2900 2650 2900 3000
+Wire Wire Line
+	2900 3000 3650 3000
+Connection ~ 3650 3000
+$Comp
+L C_Small C6
+U 1 1 5AA8EC5C
+P 6400 4650
+F 0 "C6" H 6500 4650 50  0000 L CNN
+F 1 "0.1uF" V 6300 4600 31  0000 L CNN
+F 2 "teensy:Cap_SmV" H 6400 4650 50  0001 C CNN
+F 3 "" H 6400 4650 50  0001 C CNN
+	1    6400 4650
+	1    0    0    -1
+$EndComp
+$Comp
+L GND #PWR019
+U 1 1 5AA8ED0D
+P 6400 4750
+F 0 "#PWR019" H 6400 4500 50  0001 C CNN
+F 1 "GND" H 6400 4600 50  0000 C CNN
+F 2 "" H 6400 4750 50  0001 C CNN
+F 3 "" H 6400 4750 50  0001 C CNN
+	1    6400 4750
+	1    0    0    -1
+$EndComp
+Wire Wire Line
+	6400 4550 6600 4550
+Wire Wire Line
+	6600 4550 6600 4950
+$Comp
+L Conn_01x02 J2
+U 1 1 5AA8FB22
+P 8250 4750
+F 0 "J2" H 8250 4550 50  0000 C CNN
+F 1 "Conn_01x02" H 8300 4850 50  0000 C CNN
+F 2 "teensy:Conn_Power_2" H 8250 4750 50  0001 C CNN
+F 3 "" H 8250 4750 50  0001 C CNN
+	1    8250 4750
+	1    0    0    -1
+$EndComp
+$Comp
+L GND #PWR020
+U 1 1 5AA8FBF4
+P 7550 4950
+F 0 "#PWR020" H 7550 4700 50  0001 C CNN
+F 1 "GND" H 7550 4800 50  0000 C CNN
+F 2 "" H 7550 4950 50  0001 C CNN
+F 3 "" H 7550 4950 50  0001 C CNN
+	1    7550 4950
+	1    0    0    -1
+$EndComp
+$Comp
+L C_Small C7
+U 1 1 5AA8FC2D
+P 7550 4850
+F 0 "C7" H 7650 4850 50  0000 L CNN
+F 1 "0.1uF" V 7450 4800 31  0000 L CNN
+F 2 "teensy:Cap_SmV" H 7550 4850 50  0001 C CNN
+F 3 "" H 7550 4850 50  0001 C CNN
+	1    7550 4850
+	1    0    0    -1
+$EndComp
+Wire Wire Line
+	7200 4750 8050 4750
+Connection ~ 7550 4750
+$Comp
+L GND #PWR021
+U 1 1 5AAA08CD
+P 8050 4850
+F 0 "#PWR021" H 8050 4600 50  0001 C CNN
+F 1 "GND" H 8050 4700 50  0000 C CNN
+F 2 "" H 8050 4850 50  0001 C CNN
+F 3 "" H 8050 4850 50  0001 C CNN
+	1    8050 4850
+	1    0    0    -1
+$EndComp
+Wire Wire Line
+	7200 4950 7200 4750
 $Comp
 L LCD1602A U3
-U 1 1 5A4DF8E6
+U 1 1 5AAA5D2C
 P 8250 2900
 F 0 "U3" H 7950 3700 60  0000 C CNN
 F 1 "LCD1602A" H 8250 2700 60  0000 C CNN
-F 2 "teensy:Conn_LCD16" H 8250 2900 60  0001 C CNN
+F 2 "" H 8250 2900 60  0001 C CNN
 F 3 "" H 8250 2900 60  0001 C CNN
 	1    8250 2900
 	1    0    0    -1
 $EndComp
-Wire Wire Line
-	2900 2050 4100 2050
-Wire Wire Line
-	2900 2650 2900 3000
-Wire Wire Line
-	2900 3000 3650 3000
-Connection ~ 3650 3000
+$Comp
+L Teensy3.2 U2
+U 1 1 5AAA657C
+P 5950 2950
+F 0 "U2" H 5600 3800 60  0000 C CNN
+F 1 "Teensy3.2" H 5950 2950 60  0000 C CNN
+F 2 "" H 5950 2950 60  0001 C CNN
+F 3 "" H 5950 2950 60  0001 C CNN
+	1    5950 2950
+	1    0    0    -1
+$EndComp
 $EndSCHEMATC

Commit message: Final version?
Parts:
- added D1: 1N4001, teensy:Diode_SmH, symbol Diode_SmH
- added J3: Conn_01x02, teensy:Conn_Power_2, symbol Conn_01x02-RESCUE-DigitalVFO
- added R11: 0R0, teensy:Res_SmH, symbol R_Small
- J2: symbol Conn_01x02 -> Conn_01x02-RESCUE-DigitalVFO
- SW1: symbol Rotary_Encoder_Switch -> Rotary_Encoder_Switch-RESCUE-DigitalVFO
- U1: symbol 74HC14 -> 74HC14-RESCUE-DigitalVFO
Connections:
- net +5V: now also R11.2
- net GND: now also C1.2, C2.2, C3.2, C4.2, C5.2, C6.2, C7.2, J1.2 (Ext), J2.2 (Pin_2), R10.2, R8.2, SW1.2 (C), SW1.4, U1.11, U1.13, U1.9, U2.1 (GND), U2.27 (AGND), U3.1 (Vss), U3.5 (RW), U4.5 (GND)
- net at C7.1, U4.8 (+Vin): now also D1.1 (K); no longer J2.1 (Pin_1)
- new net: D1.2 (A), J2.1 (Pin_1)
- new net: J3.1 (Pin_1), R11.1
Other:
- moved on the sheet: J2
Changed lines of the file:
@@
 $EndDescr
 $Comp
-L 74HC14 U1
+L 74HC14-RESCUE-DigitalVFO U1
 U 1 1 5A2E6497
 P 4550 2350
@@
 $EndComp
 $Comp
-L 74HC14 U1
+L 74HC14-RESCUE-DigitalVFO U1
 U 2 1 5A2E6500
 P 4100 3300
@@
 $EndComp
 $Comp
-L 74HC14 U1
+L 74HC14-RESCUE-DigitalVFO U1
 U 3 1 5A2E6525
 P 3650 4200
@@
 $EndComp
 $Comp
-L 74HC14 U1
+L 74HC14-RESCUE-DigitalVFO U1
 U 4 1 5A2E6584
 P 4400 4800
@@
 $EndComp
 $Comp
-L 74HC14 U1
+L 74HC14-RESCUE-DigitalVFO U1
 U 5 1 5A2E65B5
 P 4400 5200
@@
 $EndComp
 $Comp
-L 74HC14 U1
+L 74HC14-RESCUE-DigitalVFO U1
 U 6 1 5A2E6601
 P 4400 5600
@@
 $EndComp
 $Comp
-L Rotary_Encoder_Switch SW1
+L Rotary_Encoder_Switch-RESCUE-DigitalVFO SW1
 U 1 1 5A2E782F
 P 2800 2350
@@
 $EndComp
 $Comp
-L GND #PWR01
+L GND-RESCUE-DigitalVFO #PWR01
 U 1 1 5A2E80CF
 P 2700 2050
@@
 	6900 4600 6900 4950
 $Comp
-L GND #PWR02
+L GND-RESCUE-DigitalVFO #PWR02
 U 1 1 5A320C77
 P 4100 2650
@@
 $EndComp
 $Comp
-L GND #PWR03
+L GND-RESCUE-DigitalVFO #PWR03
 U 1 1 5A320DE5
 P 3200 4500
@@
 $EndComp
 $Comp
-L GND #PWR04
+L GND-RESCUE-DigitalVFO #PWR04
 U 1 1 5A32516D
 P 3650 3600
@@
 $EndComp
 $Comp
-L GND #PWR05
+L GND-RESCUE-DigitalVFO #PWR05
 U 1 1 5A325232
 P 2800 2650
@@
 $EndComp
 $Comp
-L GND #PWR06
+L GND-RESCUE-DigitalVFO #PWR06
 U 1 1 5A32532D
 P 6950 3200
@@
 $EndComp
 $Comp
-L GND #PWR07
+L GND-RESCUE-DigitalVFO #PWR07
 U 1 1 5A325451
 P 8350 3850
@@
 $EndComp
 $Comp
-L GND #PWR08
+L GND-RESCUE-DigitalVFO #PWR08
 U 1 1 5A325545
 P 5600 3950
@@
 $EndComp
 $Comp
-L GND #PWR09
+L GND-RESCUE-DigitalVFO #PWR09
 U 1 1 5A32580E
 P 6750 4900
@@
 $EndComp
 $Comp
-L GND #PWR010
+L GND-RESCUE-DigitalVFO #PWR010
 U 1 1 5A32593F
 P 7150 4050
@@
 $EndComp
 $Comp
-L GND #PWR011
+L GND-RESCUE-DigitalVFO #PWR011
 U 1 1 5A325A73
 P 3950 5600
@@
 $EndComp
 $Comp
-L GND #PWR012
+L GND-RESCUE-DigitalVFO #PWR012
 U 1 1 5A325F7B
 P 7100 4450
@@
 $EndComp
 $Comp
-L GND #PWR018
+L GND-RESCUE-DigitalVFO #PWR018
 U 1 1 5A3E323F
 P 6200 2000
@@
 $EndComp
 $Comp
-L GND #PWR019
+L GND-RESCUE-DigitalVFO #PWR019
 U 1 1 5AA8ED0D
 P 6400 4750
@@
 	6600 4550 6600 4950
 $Comp
-L Conn_01x02 J2
+L Conn_01x02-RESCUE-DigitalVFO J2
 U 1 1 5AA8FB22
-P 8250 4750
-F 0 "J2" H 8250 4550 50  0000 C CNN
-F 1 "Conn_01x02" H 8300 4850 50  0000 C CNN
-F 2 "teensy:Conn_Power_2" H 8250 4750 50  0001 C CNN
-F 3 "" H 8250 4750 50  0001 C CNN
-	1    8250 4750
-	1    0    0    -1
-$EndComp
-$Comp
-L GND #PWR020
+P 8500 4750
+F 0 "J2" H 8500 4550 50  0000 C CNN
+F 1 "Conn_01x02" H 8550 4850 50  0000 C CNN
+F 2 "teensy:Conn_Power_2" H 8500 4750 50  0001 C CNN
+F 3 "" H 8500 4750 50  0001 C CNN
+	1    8500 4750
+	1    0    0    -1
+$EndComp
+$Comp
+L GND-RESCUE-DigitalVFO #PWR020
 U 1 1 5AA8FBF4
 P 7550 4950
@@
 	1    0    0    -1
 $EndComp
-Wire Wire Line
-	7200 4750 8050 4750
 Connection ~ 7550 4750
 $Comp
-L GND #PWR021
+L GND-RESCUE-DigitalVFO #PWR021
 U 1 1 5AAA08CD
-P 8050 4850
-F 0 "#PWR021" H 8050 4600 50  0001 C CNN
-F 1 "GND" H 8050 4700 50  0000 C CNN
-F 2 "" H 8050 4850 50  0001 C CNN
-F 3 "" H 8050 4850 50  0001 C CNN
-	1    8050 4850
+P 8300 4850
+F 0 "#PWR021" H 8300 4600 50  0001 C CNN
+F 1 "GND" H 8300 4700 50  0000 C CNN
+F 2 "" H 8300 4850 50  0001 C CNN
+F 3 "" H 8300 4850 50  0001 C CNN
+	1    8300 4850
 	1    0    0    -1
 $EndComp
@@
 	1    0    0    -1
 $EndComp
+$Comp
+L Conn_01x02-RESCUE-DigitalVFO J3
+U 1 1 5AB4AC63
+P 8250 5650
+F 0 "J3" H 8250 5450 50  0000 C CNN
+F 1 "Conn_01x02" H 8300 5750 50  0000 C CNN
+F 2 "teensy:Conn_Power_2" H 8250 5650 50  0001 C CNN
+F 3 "" H 8250 5650 50  0001 C CNN
+	1    8250 5650
+	1    0    0    -1
+$EndComp
+$Comp
+L R_Small R11
+U 1 1 5AB4AFD4
+P 7900 5550
+F 0 "R11" V 8000 5500 50  0000 L CNN
+F 1 "0R0" V 7900 5500 31  0000 L CNN
+F 2 "teensy:Res_SmH" H 7900 5550 50  0001 C CNN
+F 3 "" H 7900 5550 50  0001 C CNN
+	1    7900 5550
+	-1   0    0    1
+$EndComp
+$Comp
+L GND #PWR022
+U 1 1 5AB4B0AA
+P 8050 5850
+F 0 "#PWR022" H 8050 5600 50  0001 C CNN
+F 1 "GND" H 8050 5700 50  0000 C CNN
+F 2 "" H 8050 5850 50  0001 C CNN
+F 3 "" H 8050 5850 50  0001 C CNN
+	1    8050 5850
+	1    0    0    -1
+$EndComp
+Wire Wire Line
+	8100 5750 8050 5750
+Wire Wire Line
+	8050 5750 8050 5850
+$Comp
+L Diode_SmH D1
+U 1 1 5AB4C080
+P 8000 4750
+F 0 "D1" H 7950 4830 50  0000 L CNN
+F 1 "1N4001" H 7850 4670 50  0000 L CNN
+F 2 "teensy:Diode_SmH" V 8000 4750 50  0001 C CNN
+F 3 "" V 8000 4750 50  0001 C CNN
+	1    8000 4750
+	1    0    0    -1
+$EndComp
+Wire Wire Line
+	7200 4750 7900 4750
+Wire Wire Line
+	8100 4750 8300 4750
+$Comp
+L +5V #PWR023
+U 1 1 5AB4C4B9
+P 7900 5450
+F 0 "#PWR023" H 7900 5300 50  0001 C CNN
+F 1 "+5V" H 7900 5590 50  0000 C CNN
+F 2 "" H 7900 5450 50  0001 C CNN
+F 3 "" H 7900 5450 50  0001 C CNN
+	1    7900 5450
+	1    0    0    -1
+$EndComp
+Wire Wire Line
+	7900 5650 8050 5650
 $EndSCHEMATC
