File: kicad/DigitalVFO.sch (KiCad schematic (older format))
At the start: 28 parts, among them J1 RF Out, J2 Battery, J3 SW_LED, Q1 2N2222A, SW1 Rotary_Encoder_Switch, U1 74HC14, U2 Teensy3.2, U3 LCD1602A, U4 DDS-60

Commit message: Version 1.4
Parts:
- added C8: 0.1uF, DigitalVFO:Cap_SmV, symbol C_Small
- added R12: 39K, DigitalVFO:Res_SmH, symbol R_Small
- added R13: 10K, DigitalVFO:Res_SmH, symbol R_Small
- J1: footprint DigitalVFO:BNC_Socket -> DigitalVFO:BNC_Socket_TYCO-AMP
- U2: footprint DigitalVFO:Conn_DIP28w -> (none)
Connections:
- net GND: now also C8.2, R13.2
- net at D1.2 (A), J2.1 (Pin_1): now also R12.1
- net at U2.21 (19): now also C8.1, R12.2, R13.1
Other:
- note added: "Optional external battery and\nmonitoring circuit, plus\npower switch with LED.\nVFO can be run from USB\npower from Teensy 3.2."
- note removed: "Optional external battery\nand power switch with LED.\nVFO can be run from USB\npower from Teensy 3.2."
- moved on the sheet: D1
Changed lines of the file:
@@
 Sheet 1 1
 Title "DigitalVFO"
-Date "26 March 2018"
-Rev "1.2"
+Date "27 April 2018"
+Rev "1.4"
 Comp ""
 Comment1 "Provision for internal battery and power switch with LED."
-Comment2 "A VFO controlled by a rotary encoder with push switch."
+Comment2 "Teensy can monitor input Lithium battery voltage."
 Comment3 ""
-Comment4 ""
+Comment4 "A VFO controlled by a rotary encoder."
 $EndDescr
 $Comp
@@
 L D_ALT D1
 U 1 1 5AB7F8C6
-P 8550 4400
-F 0 "D1" H 8550 4500 50  0000 C CNN
-F 1 "1N4001" H 8550 4300 50  0000 C CNN
-F 2 "DigitalVFO:Diode_SmH" H 8550 4400 50  0001 C CNN
-F 3 "" H 8550 4400 50  0001 C CNN
-	1    8550 4400
+P 8250 4400
+F 0 "D1" H 8250 4500 50  0000 C CNN
+F 1 "1N4001" H 8250 4300 50  0000 C CNN
+F 2 "DigitalVFO:Diode_SmH" H 8250 4400 50  0001 C CNN
+F 3 "" H 8250 4400 50  0001 C CNN
+	1    8250 4400
 	1    0    0    -1
 $EndComp
@@
 $EndComp
 Wire Wire Line
-	8700 4400 8900 4400
-Wire Wire Line
-	8400 4400 7450 4400
+	8900 4400 8400 4400
+Wire Wire Line
+	8100 4400 7450 4400
 Wire Wire Line
 	7450 4400 7450 5250
@@
 	8900 4500 8900 4650
 $Comp
-L Teensy3.2 U2
-U 1 1 5AB80DEC
-P 5500 2250
-F 0 "U2" H 4950 3400 60  0000 C CNN
-F 1 "Teensy3.2" H 5500 2250 60  0000 C CNN
-F 2 "DigitalVFO:Conn_DIP28w" H 5500 2250 60  0001 C CNN
-F 3 "" H 5500 2250 60  0001 C CNN
-	1    5500 2250
-	1    0    0    -1
-$EndComp
-$Comp
 L DDS-60 U4
 U 1 1 5AB80E84
@@
 F 0 "J1" H 6930 4460 50  0000 C CNN
 F 1 "RF Out" H 7050 4600 50  0000 C CNN
-F 2 "DigitalVFO:BNC_Socket" V 7050 4450 50  0001 C CNN
+F 2 "DigitalVFO:BNC_Socket_TYCO-AMP" V 7050 4450 50  0001 C CNN
 F 3 "" V 7050 4450 50  0001 C CNN
 	1    7050 4450
@@
 $EndComp
 Wire Notes Line
-	7350 4200 9450 4200
-Wire Notes Line
-	9450 4200 9450 6150
+	9450 3800 9450 6150
 Wire Notes Line
 	9450 6150 8150 6150
@@
 	8150 5250 7350 5250
 Wire Notes Line
-	7350 5250 7350 4200
+	7350 5250 7350 3800
 Text Notes 9550 4550 0    60   ~ 0
-Optional external battery\nand power switch with LED.\nVFO can be run from USB\npower from Teensy 3.2.
+Optional external battery and\nmonitoring circuit, plus\npower switch with LED.\nVFO can be run from USB\npower from Teensy 3.2.
 $Bitmap
 Pos 10900 6850
@@
 EndData
 $EndBitmap
+Wire Notes Line
+	7350 3800 9450 3800
+$Comp
+L R_Small R12
+U 1 1 5AE2892A
+P 8100 3900
+F 0 "R12" V 8200 3850 50  0000 L CNN
+F 1 "39K" V 8050 4000 50  0000 L CNN
+F 2 "DigitalVFO:Res_SmH" H 8100 3900 50  0001 C CNN
+F 3 "" H 8100 3900 50  0001 C CNN
+	1    8100 3900
+	0    1    1    0
+$EndComp
+$Comp
+L R_Small R13
+U 1 1 5AE28A8A
+P 7700 3900
+F 0 "R13" V 7800 3850 50  0000 L CNN
+F 1 "10K" V 7650 3650 50  0000 L CNN
+F 2 "DigitalVFO:Res_SmH" H 7700 3900 50  0001 C CNN
+F 3 "" H 7700 3900 50  0001 C CNN
+	1    7700 3900
+	0    1    1    0
+$EndComp
+Wire Wire Line
+	7800 3900 8000 3900
+Wire Wire Line
+	8200 3900 8900 3900
+Wire Wire Line
+	8900 3900 8900 4400
+Connection ~ 8900 4400
+$Comp
+L C_Small C8
+U 1 1 5AE28C83
+P 7900 4050
+F 0 "C8" H 7910 4120 50  0000 L CNN
+F 1 "0.1uF" H 7910 3970 50  0000 L CNN
+F 2 "DigitalVFO:Cap_SmV" H 7900 4050 50  0001 C CNN
+F 3 "" H 7900 4050 50  0001 C CNN
+	1    7900 4050
+	1    0    0    -1
+$EndComp
+Wire Wire Line
+	7900 2100 7900 3950
+Connection ~ 7900 3900
+$Comp
+L GND #PWR028
+U 1 1 5AE28DCB
+P 7900 4150
+F 0 "#PWR028" H 7900 3900 50  0001 C CNN
+F 1 "GND" H 7900 4000 50  0000 C CNN
+F 2 "" H 7900 4150 50  0001 C CNN
+F 3 "" H 7900 4150 50  0001 C CNN
+	1    7900 4150
+	1    0    0    -1
+$EndComp
+$Comp
+L GND #PWR029
+U 1 1 5AE290F2
+P 7500 4000
+F 0 "#PWR029" H 7500 3750 50  0001 C CNN
+F 1 "GND" H 7500 3850 50  0000 C CNN
+F 2 "" H 7500 4000 50  0001 C CNN
+F 3 "" H 7500 4000 50  0001 C CNN
+	1    7500 4000
+	1    0    0    -1
+$EndComp
+Wire Wire Line
+	7500 4000 7500 3900
+Wire Wire Line
+	7500 3900 7600 3900
+Wire Wire Line
+	7900 2100 6300 2100
+$Comp
+L Teensy3.2 U2
+U 1 1 5AE2B0F8
+P 5500 2250
+F 0 "U2" H 4950 3400 60  0000 C CNN
+F 1 "Teensy3.2" H 5500 2250 60  0000 C CNN
+F 2 "" H 5500 2250 60  0001 C CNN
+F 3 "" H 5500 2250 60  0001 C CNN
+	1    5500 2250
+	1    0    0    -1
+$EndComp
 $EndSCHEMATC

Commit message: v1.5 - more compact layout
Parts:
- R12: value 39K -> 22K
- SW1: value Rotary_Encoder_Switch -> Rotary_Encoder
Changed lines of the file:
@@
 P 1550 1500
 F 0 "SW1" V 1700 1200 50  0000 C CNN
-F 1 "Rotary_Encoder_Switch" H 1600 1800 50  0000 C CNN
+F 1 "Rotary_Encoder" H 1600 1800 50  0000 C CNN
 F 2 "DigitalVFO:Conn_RE_Switch" H 1450 1660 50  0001 C CNN
 F 3 "" H 1550 1760 50  0001 C CNN
@@
 L GND #PWR016
 U 1 1 5AB7F12E
-P 9100 3550
-F 0 "#PWR016" H 9100 3300 50  0001 C CNN
-F 1 "GND" H 9100 3400 50  0000 C CNN
-F 2 "" H 9100 3550 50  0001 C CNN
-F 3 "" H 9100 3550 50  0001 C CNN
-	1    9100 3550
+P 8600 3550
+F 0 "#PWR016" H 8600 3300 50  0001 C CNN
+F 1 "GND" H 8600 3400 50  0000 C CNN
+F 2 "" H 8600 3550 50  0001 C CNN
+F 3 "" H 8600 3550 50  0001 C CNN
+	1    8600 3550
 	1    0    0    -1
 $EndComp
@@
 P 8100 3900
 F 0 "R12" V 8200 3850 50  0000 L CNN
-F 1 "39K" V 8050 4000 50  0000 L CNN
+F 1 "22K" V 8050 4000 50  0000 L CNN
 F 2 "DigitalVFO:Res_SmH" H 8100 3900 50  0001 C CNN
 F 3 "" H 8100 3900 50  0001 C CNN
@@
 	1    0    0    -1
 $EndComp
+Connection ~ 3200 800
+Connection ~ 5000 3550
+Connection ~ 8600 3550
 $EndSCHEMATC

Commit message: Added testpoints and 1602A mount holes
Connections:
- net BATT: now reaches C7.1, D1.1 (K), U4.8 (+Vin)
- net RF: now reaches J1.1 (In), U4.6 (RF_out)
- net BMON: now reaches C8.1, R12.2, R13.1, U2.21 (19)
Changed lines of the file:
@@
 Title "DigitalVFO"
 Date "27 April 2018"
-Rev "1.4"
+Rev "1.5"
 Comp ""
 Comment1 "Provision for internal battery and power switch with LED."
-Comment2 "Teensy can monitor input Lithium battery voltage."
+Comment2 "Microcontroller can monitor input Lithium battery voltage."
 Comment3 ""
-Comment4 "A VFO controlled by a rotary encoder."
+Comment4 "A DDS VFO controlled by a rotary encoder."
 $EndDescr
 $Comp
@@
 	2450 2400 2450 2500
 Wire Wire Line
-	3200 800  9100 800
-Wire Wire Line
-	5500 800  5500 950
+	3200 750  9100 750
+Wire Wire Line
+	5500 750  5500 950
 $Comp
 L +5V #PWR011
 U 1 1 5AB7D64D
-P 3200 800
-F 0 "#PWR011" H 3200 650 50  0001 C CNN
-F 1 "+5V" H 3200 940 50  0000 C CNN
-F 2 "" H 3200 800 50  0001 C CNN
-F 3 "" H 3200 800 50  0001 C CNN
-	1    3200 800
+P 3200 750
+F 0 "#PWR011" H 3200 600 50  0001 C CNN
+F 1 "+5V" H 3200 890 50  0000 C CNN
+F 2 "" H 3200 750 50  0001 C CNN
+F 3 "" H 3200 750 50  0001 C CNN
+	1    3200 750
 	1    0    0    -1
 $EndComp
@@
 	6450 4850 6650 4850
 Wire Wire Line
-	9100 800  9100 950
-Connection ~ 5500 800
-Wire Wire Line
-	8600 950  8600 800
-Connection ~ 8600 800
+	9100 750  9100 950
+Connection ~ 5500 750
+Wire Wire Line
+	8600 950  8600 750
+Connection ~ 8600 750
 Wire Wire Line
 	8600 3550 9100 3550
@@
 $EndComp
 Wire Wire Line
-	6700 850  6700 800
-Connection ~ 6700 800
+	6700 850  6700 750
+Connection ~ 6700 750
 Wire Wire Line
 	6700 1050 6700 1100
@@
 L VCC #PWR022
 U 1 1 5AB7EED1
-P 8600 800
-F 0 "#PWR022" H 8600 650 50  0001 C CNN
-F 1 "VCC" H 8600 950 50  0000 C CNN
-F 2 "" H 8600 800 50  0001 C CNN
-F 3 "" H 8600 800 50  0001 C CNN
-	1    8600 800
+P 8600 750
+F 0 "#PWR022" H 8600 600 50  0001 C CNN
+F 1 "VCC" H 8600 900 50  0000 C CNN
+F 2 "" H 8600 750 50  0001 C CNN
+F 3 "" H 8600 750 50  0001 C CNN
+	1    8600 750
 	1    0    0    -1
 $EndComp
@@
 L PWR_FLAG #FLG023
 U 1 1 5AB8A9A8
-P 3300 5850
-F 0 "#FLG023" H 3300 5925 50  0001 C CNN
-F 1 "PWR_FLAG" H 3300 6000 50  0000 C CNN
-F 2 "" H 3300 5850 50  0001 C CNN
-F 3 "" H 3300 5850 50  0001 C CNN
-	1    3300 5850
+P 3250 5850
+F 0 "#FLG023" H 3250 5925 50  0001 C CNN
+F 1 "PWR_FLAG" H 3250 6000 50  0000 C CNN
+F 2 "" H 3250 5850 50  0001 C CNN
+F 3 "" H 3250 5850 50  0001 C CNN
+	1    3250 5850
 	1    0    0    -1
 $EndComp
@@
 L GND #PWR024
 U 1 1 5AB8A9FE
-P 3300 5950
-F 0 "#PWR024" H 3300 5700 50  0001 C CNN
-F 1 "GND" H 3300 5800 50  0000 C CNN
-F 2 "" H 3300 5950 50  0001 C CNN
-F 3 "" H 3300 5950 50  0001 C CNN
-	1    3300 5950
-	1    0    0    -1
-$EndComp
-Wire Wire Line
-	3300 5850 3300 5950
+P 3250 5950
+F 0 "#PWR024" H 3250 5700 50  0001 C CNN
+F 1 "GND" H 3250 5800 50  0000 C CNN
+F 2 "" H 3250 5950 50  0001 C CNN
+F 3 "" H 3250 5950 50  0001 C CNN
+	1    3250 5950
+	1    0    0    -1
+$EndComp
+Wire Wire Line
+	3250 5850 3250 5950
 $Comp
 L PWR_FLAG #FLG025
@@
 	1    0    0    -1
 $EndComp
-Connection ~ 3200 800
+Connection ~ 3200 750
 Connection ~ 5000 3550
 Connection ~ 8600 3550
+Wire Wire Line
+	3200 750  3200 800
+Text Label 7650 2100 0    60   ~ 0
+BMON
+Text Label 7050 4900 0    60   ~ 0
+RF
+Text Label 7450 4600 0    60   ~ 0
+BATT
 $EndSCHEMATC
