File: kicad/DigitalVFO.sch (KiCad schematic (older format))
At the start: 31 parts, among them J1 RF Out, J2 Battery, J3 SW_LED, Q1 2N2222A, SW1 Rotary_Encoder, U1 74HC14, U2 Teensy3.2, U3 LCD1602A, U4 DDS-60

Commit message: Updated the PCB
Parts:
- C1, C2, C3, C5, C6, C7, C8: symbol C_Small -> DigitalVFO:C_Small
- C4: symbol CP_Small -> DigitalVFO:CP_Small
- D1: symbol D_ALT -> DigitalVFO:D_ALT
- J1: symbol Conn_Coaxial -> DigitalVFO:Conn_Coaxial
- J2, J3: symbol Conn_01x02 -> DigitalVFO:Conn_01x02
- Q1: symbol Q_NPN_EBC -> DigitalVFO:Q_NPN_EBC
- R1, R10, R11, R12, R13, R2, R3, R4, R5, R6, R7, R8, R9: symbol R_Small -> DigitalVFO:R_Small
- SW1: symbol Rotary_Encoder_Switch -> DigitalVFO:Rotary_Encoder_Switch
- U1: symbol 74HC14 -> DigitalVFO:74HC14
- U2: symbol Teensy3.2 -> DigitalVFO:Teensy3.2
- U3: symbol LCD1602A -> DigitalVFO:LCD1602A
- U4: symbol DDS-60 -> DigitalVFO:DDS-60

Commit message: Small changes
Parts:
- C1, C2, C3, C5, C6, C7, C8: symbol DigitalVFO:C_Small -> DigitalVFO-rescue:C_Small-DigitalVFO
- C4: symbol DigitalVFO:CP_Small -> DigitalVFO-rescue:CP_Small-DigitalVFO
- D1: symbol DigitalVFO:D_ALT -> DigitalVFO-rescue:D_ALT-DigitalVFO
- J1: symbol DigitalVFO:Conn_Coaxial -> DigitalVFO-rescue:Conn_Coaxial-DigitalVFO
- J2, J3: symbol DigitalVFO:Conn_01x02 -> DigitalVFO-rescue:Conn_01x02-DigitalVFO
- Q1: symbol DigitalVFO:Q_NPN_EBC -> DigitalVFO-rescue:Q_NPN_EBC-DigitalVFO
- R1, R10, R11, R12, R13, R2, R3, R4, R5, R6, R7, R8, R9: symbol DigitalVFO:R_Small -> DigitalVFO-rescue:R_Small-DigitalVFO
- SW1: symbol DigitalVFO:Rotary_Encoder_Switch -> DigitalVFO-rescue:Rotary_Encoder_Switch-DigitalVFO
- U1: symbol DigitalVFO:74HC14 -> DigitalVFO-rescue:74HC14-DigitalVFO
- U2: symbol DigitalVFO:Teensy3.2 -> DigitalVFO-rescue:Teensy3.2-DigitalVFO
- U3: symbol DigitalVFO:LCD1602A -> DigitalVFO-rescue:LCD1602A-DigitalVFO
- U4: symbol DigitalVFO:DDS-60 -> DigitalVFO-rescue:DDS-60-DigitalVFO
Changed lines of the file:
@@
 $EndDescr
 $Comp
-L DigitalVFO:74HC14 U1
+L DigitalVFO-rescue:74HC14-DigitalVFO U1
 U 1 1 5AB77F50
 P 4000 1350
@@
 $EndComp
 $Comp
-L DigitalVFO:74HC14 U1
+L DigitalVFO-rescue:74HC14-DigitalVFO U1
 U 2 1 5AB77F8D
 P 3250 2150
@@
 $EndComp
 $Comp
-L DigitalVFO:74HC14 U1
+L DigitalVFO-rescue:74HC14-DigitalVFO U1
 U 3 1 5AB77FD8
 P 2550 2950
@@
 $EndComp
 $Comp
-L DigitalVFO:74HC14 U1
+L DigitalVFO-rescue:74HC14-DigitalVFO U1
 U 4 1 5AB7800C
 P 1800 4850
@@
 $EndComp
 $Comp
-L DigitalVFO:74HC14 U1
+L DigitalVFO-rescue:74HC14-DigitalVFO U1
 U 5 1 5AB78036
 P 1800 5250
@@
 $EndComp
 $Comp
-L DigitalVFO:74HC14 U1
+L DigitalVFO-rescue:74HC14-DigitalVFO U1
 U 6 1 5AB78082
 P 1800 5650
@@
 $EndComp
 $Comp
-L DigitalVFO:Rotary_Encoder_Switch SW1
+L DigitalVFO-rescue:Rotary_Encoder_Switch-DigitalVFO SW1
 U 1 1 5AB790E1
 P 1550 1500
@@
 $EndComp
 $Comp
-L DigitalVFO:Q_NPN_EBC Q1
+L DigitalVFO-rescue:Q_NPN_EBC-DigitalVFO Q1
 U 1 1 5AB79125
 P 7050 3150
@@
 	6300 1850 8050 1850
 $Comp
-L DigitalVFO:R_Small R7
+L DigitalVFO-rescue:R_Small-DigitalVFO R7
 U 1 1 5AB7A839
 P 6550 3150
@@
 	6650 3150 6800 3150
 $Comp
-L DigitalVFO:LCD1602A U3
+L DigitalVFO-rescue:LCD1602A-DigitalVFO U3
 U 1 1 5AB7B041
 P 8850 2250
@@
 	7100 2900 8050 2900
 $Comp
-L DigitalVFO:R_Small R8
+L DigitalVFO-rescue:R_Small-DigitalVFO R8
 U 1 1 5AB7B0A8
 P 7100 3550
@@
 	7100 3650 7100 3750
 $Comp
-L DigitalVFO:C_Small C6
+L DigitalVFO-rescue:C_Small-DigitalVFO C6
 U 1 1 5AB7B2BD
 P 6450 5000
@@
 Connection ~ 6650 4850
 $Comp
-L DigitalVFO:R_Small R9
+L DigitalVFO-rescue:R_Small-DigitalVFO R9
 U 1 1 5AB7B3DF
 P 6650 2350
@@
 $EndComp
 $Comp
-L DigitalVFO:CP_Small C4
+L DigitalVFO-rescue:CP_Small-DigitalVFO C4
 U 1 1 5AB7B49C
 P 6950 2500
@@
 $EndComp
 $Comp
-L DigitalVFO:R_Small R10
+L DigitalVFO-rescue:R_Small-DigitalVFO R10
 U 1 1 5AB7B4F4
 P 7300 2500
@@
 	6750 2350 6950 2350
 $Comp
-L DigitalVFO:R_Small R1
+L DigitalVFO-rescue:R_Small-DigitalVFO R1
 U 1 1 5AB7C67F
 P 3200 900
@@
 $EndComp
 $Comp
-L DigitalVFO:R_Small R2
+L DigitalVFO-rescue:R_Small-DigitalVFO R2
 U 1 1 5AB7C6C8
 P 3200 1200
@@
 $EndComp
 $Comp
-L DigitalVFO:C_Small C1
+L DigitalVFO-rescue:C_Small-DigitalVFO C1
 U 1 1 5AB7C723
 P 3200 1500
@@
 	3200 1600 3200 1700
 $Comp
-L DigitalVFO:R_Small R5
+L DigitalVFO-rescue:R_Small-DigitalVFO R5
 U 1 1 5AB7CFD2
 P 1750 2500
@@
 $EndComp
 $Comp
-L DigitalVFO:R_Small R6
+L DigitalVFO-rescue:R_Small-DigitalVFO R6
 U 1 1 5AB7CFD8
 P 1750 2800
@@
 $EndComp
 $Comp
-L DigitalVFO:C_Small C3
+L DigitalVFO-rescue:C_Small-DigitalVFO C3
 U 1 1 5AB7CFDE
 P 1750 3100
@@
 	1750 3200 1750 3300
 $Comp
-L DigitalVFO:R_Small R3
+L DigitalVFO-rescue:R_Small-DigitalVFO R3
 U 1 1 5AB7D0D7
 P 2450 1700
@@
 $EndComp
 $Comp
-L DigitalVFO:R_Small R4
+L DigitalVFO-rescue:R_Small-DigitalVFO R4
 U 1 1 5AB7D0DD
 P 2450 2000
@@
 $EndComp
 $Comp
-L DigitalVFO:C_Small C2
+L DigitalVFO-rescue:C_Small-DigitalVFO C2
 U 1 1 5AB7D0E3
 P 2450 2300
@@
 $EndComp
 $Comp
-L DigitalVFO:Conn_01x02 J2
+L DigitalVFO-rescue:Conn_01x02-DigitalVFO J2
 U 1 1 5AB7F850
 P 9100 4450
@@
 $EndComp
 $Comp
-L DigitalVFO:D_ALT D1
+L DigitalVFO-rescue:D_ALT-DigitalVFO D1
 U 1 1 5AB7F8C6
 P 8250 4400
@@
 $EndComp
 $Comp
-L DigitalVFO:C_Small C7
+L DigitalVFO-rescue:C_Small-DigitalVFO C7
 U 1 1 5AB7F925
 P 7750 4850
@@
 	8900 4500 8900 4650
 $Comp
-L DigitalVFO:DDS-60 U4
+L DigitalVFO-rescue:DDS-60-DigitalVFO U4
 U 1 1 5AB80E84
 P 6550 5850
@@
 $EndComp
 $Comp
-L DigitalVFO:Conn_01x02 J3
+L DigitalVFO-rescue:Conn_01x02-DigitalVFO J3
 U 1 1 5AB813E8
 P 9000 5800
@@
 $EndComp
 $Comp
-L DigitalVFO:R_Small R11
+L DigitalVFO-rescue:R_Small-DigitalVFO R11
 U 1 1 5AB81514
 P 8500 5600
@@
 	7750 4950 7750 5050
 $Comp
-L DigitalVFO:C_Small C5
+L DigitalVFO-rescue:C_Small-DigitalVFO C5
 U 1 1 5AB87925
 P 6700 950
@@
 	6700 1050 6700 1100
 $Comp
-L DigitalVFO:Conn_Coaxial J1
+L DigitalVFO-rescue:Conn_Coaxial-DigitalVFO J1
 U 1 1 5AB8824F
 P 7050 4450
@@
 	7350 3800 9450 3800
 $Comp
-L DigitalVFO:R_Small R12
+L DigitalVFO-rescue:R_Small-DigitalVFO R12
 U 1 1 5AE2892A
 P 8100 3900
@@
 $EndComp
 $Comp
-L DigitalVFO:R_Small R13
+L DigitalVFO-rescue:R_Small-DigitalVFO R13
 U 1 1 5AE28A8A
 P 7700 3900
@@
 Connection ~ 8900 4400
 $Comp
-L DigitalVFO:C_Small C8
+L DigitalVFO-rescue:C_Small-DigitalVFO C8
 U 1 1 5AE28C83
 P 7900 4050
@@
 	7500 3900 7600 3900
 $Comp
-L DigitalVFO:Teensy3.2 U2
+L DigitalVFO-rescue:Teensy3.2-DigitalVFO U2
 U 1 1 5AE2B0F8
 P 5500 2250
